Commit message: save point

File: App/Indy7/indy7_v2.urdf (robot description, URDF)
Before this commit: robot indy, 9 links, 8 joints
Links:
- link link0: mass 1.6703078 -> 1.66957888
- link link1: mass 11.44444535 -> 11.43955917
- link link2: mass 5.84766553 -> 6.11383823
- link link3: mass 2.68206064 -> 2.68211719
- link link4: mass 2.12987371 -> 2.12830848
- link link5: mass 2.22412271 -> 2.32413397
- link link6: mass 0.38254932 -> 0.39652271
- link tcp: mass 0.7 -> None
Joints:
- joint joint1: origin xyz=0                          -0.109                          0.222 rpy=1.570796327                         1.570796327                         0 -> xyz=0                          -0.109                          0.222 rpy=1.570796327                         0                         0
- joint joint2: origin xyz=-0.45                          0                          -0.0305 rpy=0                         0                         0 -> xyz=0                          0.45                          -0.0305 rpy=0                         0                         3.1415926536
- joint joint3: origin xyz=-0.267                          0                          -0.075 rpy=-1.570796327                         0                         1.570796327 -> xyz=0                          -0.267                          -0.075 rpy=-1.570796327                         0                         3.1415926536
- joint joint4: origin xyz=0                          -0.114                          0.083 rpy=1.570796327                         1.570796327                         0 -> xyz=0                          -0.114                          0.0835 rpy=1.570796327                         0                         0
- joint joint5: origin xyz=-0.168                          0                          0.069 rpy=-1.570796327                         0                         1.570796327 -> xyz=0                          0.052                          0.085 rpy=-1.570796327                         0                         0
- joint tcp: origin xyz=0.0                          0.0                          0.06 rpy=0.0                         0.0                         0.0 -> xyz=0.0                          0.0                          0.057 rpy=0.0                         0.0                         0.0
