Commit message: remove csv from tracking

File: App/Indy7/indy7.urdf (robot description, URDF)
Before this commit: robot indy, 9 links, 8 joints
Links:
- link link3: mass 2.8206064 -> 2.68206064
- link link5: mass 2.42412271 -> 2.22412271
- link link6: mass 0.28 -> 0.38254932

Commit message: [chore] : ros2 working, chore indy7 change

File: App/Indy7/indy7.urdf (robot description, URDF)
Before this commit: robot indy, 9 links, 8 joints
Links:
- link tcp: mass None -> 0.0

Commit message: unstable tunning, stable plotting, Added SetRefTcp

File: App/Indy7/indy7.urdf (robot description, URDF)
Before this commit: robot indy, 9 links, 8 joints
Links:
- link tcp: mass 0.0 -> 0.01

Commit message: 2026_05_17

File: App/Indy7/indy7.urdf (robot description, URDF)
Before this commit: robot indy, 9 links, 8 joints
Links:
- link tcp: mass 0.7 -> 0.0
