Commit message: URDF: model the real end-of-arm payload (RFT76-HA01 + tag plate, 285 g)
Measured on the robot: RFT76-HA01 F/T sensor (D76x17, 200 g) bolted straight
to the flange, metal tag plate D90x5 (~85 g Al estimate), total stack 18.5 mm.
CoM placed from the hand-eye eMo solve: flange face at z=-0.071 in the tcp
frame -> composite CoM at z=-0.060. This unmodeled mass was the driver of the
grav-comp sink and part of the CTC droop at extended poses.

Co-Authored-By: Claude Fable 5 <noreply@anthropic.com>

File: App/Indy7/indy7.urdf (robot description, URDF)
Before this commit: robot indy, 9 links, 8 joints
Links:
- link tcp: mass 0.0 -> 0.285

Commit message: A/B: remove the 285 g F/T payload from the URDF (back to zero-mass tcp)
The payload rested on a guessed tag-plate mass and on the -X tool-axis
reading that the 07-29 field check contradicted (+Z) — so grav-comp may
be pulling the wrist wrong in both magnitude and direction. Field
evidence points that way: first landings come in HIGH (banana #23 first
miss +36 mm, wrist-pitch stuck 10 deg short into the 0.15 rad settle
leash). Kinematics untouched — fk_replay output on the banana DataLog is
byte-identical, so the hand-eye calib, reach map and all plots stay
valid. Restore: git checkout 9dc5ae3 -- App/Indy7/indy7.urdf

Co-Authored-By: Claude Opus 5 <noreply@anthropic.com>

File: App/Indy7/indy7.urdf (robot description, URDF)
Before this commit: robot indy, 9 links, 8 joints
Links:
- link tcp: mass 0.285 -> 0.0
